Commit message: ros_robot

File: urdf/mrobot.urdf (robot description, URDF)
Before this commit: robot None, 0 links, 0 joints
Links:
- added link base_footprint; visual box size=0.001 0.001 0.001
- added link base_link, mass 2; collision cylinder length=0.005 radius=0.13; visual cylinder length=0.005 radius=0.13
- added link front_caster_link, mass 0.001; collision sphere radius=0.0165; visual sphere radius=0.0165
- added link left_motor, mass 0.1; collision cylinder length=0.08 radius=0.02; visual cylinder length=0.08 radius=0.02
- added link left_wheel_link, mass 0.01; collision cylinder length=0.017 radius=0.033; visual cylinder length=0.017 radius=0.033
- added link plate_1_link, mass 0.1; collision cylinder length=0.005 radius=0.13; visual cylinder length=0.005 radius=0.13
- added link plate_2_link, mass 0.01; collision cylinder length=0.005 radius=0.13; visual cylinder length=0.005 radius=0.13
- added link right_motor, mass 0.1; collision cylinder length=0.08 radius=0.02; visual cylinder length=0.08 radius=0.02
- added link right_wheel_link, mass 0.01; collision cylinder length=0.017 radius=0.033; visual cylinder length=0.017 radius=0.033
- added link standoff_2in_1_link, mass 0.001; collision box size=0.01 0.01 0.07; visual box size=0.01 0.01 0.07
- added link standoff_2in_2_link, mass 0.001; collision box size=0.01 0.01 0.07; visual box size=0.01 0.01 0.07
- added link standoff_2in_3_link, mass 0.001; collision box size=0.01 0.01 0.07; visual box size=0.01 0.01 0.07
- added link standoff_2in_4_link, mass 0.001; collision box size=0.01 0.01 0.07; visual box size=0.01 0.01 0.07
- added link standoff_2in_5_link, mass 0.001; collision box size=0.01 0.01 0.07; visual box size=0.01 0.01 0.07
- added link standoff_2in_6_link, mass 0.001; collision box size=0.01 0.01 0.07; visual box size=0.01 0.01 0.07
- added link standoff_2in_7_link, mass 0.001; collision box size=0.01 0.01 0.07; visual box size=0.01 0.01 0.07
- added link standoff_2in_8_link, mass 0.001; collision box size=0.01 0.01 0.07; visual box size=0.01 0.01 0.07
Joints:
- added joint base_footprint_joint: type fixed, parent base_footprint, child base_link, origin xyz=0 0 0.033 rpy=0 0 0
- added joint base_left_motor_joint: type fixed, parent base_link, child left_motor, origin xyz=-0.055 0.075 0 rpy=0 0 0
- added joint base_right_motor_joint: type fixed, parent base_link, child right_motor, origin xyz=-0.055 -0.075 0 rpy=0 0 0
- added joint front_caster_joint: type fixed, parent base_link, child front_caster_link, origin xyz=0.1135 0 -0.0165 rpy=0 0 0
- added joint left_wheel_joint: type continuous, parent left_motor, child left_wheel_link, origin xyz=0 0.0485 0 rpy=0 0 0, axis 0 1 0
- added joint plate_1_joint: type fixed, parent base_link, child plate_1_link, origin xyz=0 0 0.07 rpy=0 0 0
- added joint plate_2_joint: type fixed, parent plate_1_link, child plate_2_link, origin xyz=0 0 0.07 rpy=0 0 0
- added joint right_wheel_joint: type continuous, parent right_motor, child right_wheel_link, origin xyz=0 -0.0485 0 rpy=0 0 0, axis 0 1 0
- added joint standoff_2in_1_joint: type fixed, parent base_link, child standoff_2in_1_link, origin xyz=-0.09 -0.07 0.035 rpy=0 0 0
- added joint standoff_2in_2_joint: type fixed, parent base_link, child standoff_2in_2_link, origin xyz=-0.09 0.07 0.035 rpy=0 0 0
- added joint standoff_2in_3_joint: type fixed, parent base_link, child standoff_2in_3_link, origin xyz=0.06 -0.1 0.035 rpy=0 0 0
- added joint standoff_2in_4_joint: type fixed, parent base_link, child standoff_2in_4_link, origin xyz=0.06 0.1 0.035 rpy=0 0 0
- added joint standoff_2in_5_joint: type fixed, parent standoff_2in_1_link, child standoff_2in_5_link, origin xyz=0 0 0.07 rpy=0 0 0
- added joint standoff_2in_6_joint: type fixed, parent standoff_2in_2_link, child standoff_2in_6_link, origin xyz=0 0 0.07 rpy=0 0 0
- added joint standoff_2in_7_joint: type fixed, parent standoff_2in_3_link, child standoff_2in_7_link, origin xyz=0 0 0.07 rpy=0 0 0
- added joint standoff_2in_8_joint: type fixed, parent standoff_2in_4_link, child standoff_2in_8_link, origin xyz=0 0 0.07 rpy=0 0 0
